File: PHMKeychain.kicad_sch (KiCad schematic)
At the start: 12 parts, among them J1 Conn_02x03_Odd_Even, Q1 HL2301A, U1 ATTINY85-20SU_C31540447

Commit message: Organized
Parts:
- removed J1: Conn_02x03_Odd_Even, Connector_PinHeader_1.00mm:PinHeader_1x06_P1.00mm_Vertical, symbol Connector_Generic:Conn_02x03_Odd_Even
- added J1: Conn_01x06, Connector_PinHeader_2.54mm:PinHeader_1x06_P2.54mm_Vertical, symbol Connector_Generic:Conn_01x06
- S1: value Tactile Button, 160gf -> Tactile Button
Connections:
- net GND: now also J1.6 (Pin_6)
- net MISO: now also J1.1 (Pin_1)
- net RESET: now also J1.5 (Pin_5)
- net SCK: now also J1.3 (Pin_3)
- net VCC: now also J1.2 (Pin_2)
- net at C3.1: now also U1.3 (PB4); no longer LS1.1 (LEAD+)
- net at C3.2: now also LS1.1 (LEAD+); no longer U1.3 (PB4)
- net MOSI / LATCH renamed LATCH
- net LATCH: now also J1.4 (Pin_4)
- no-connect marks 0 -> 1
Other:
- note added: "ATTiny85 + Speaker + LowPassFilterCap"
- note added: "Connectors"
- note added: "Coupling Capacitors"
- note added: "Power + Latch"
- note added: "Power LED"
- moved on the sheet: BT1, C1, C2, C3, D1, LS1, Q1, R1, R2, S1

Commit message: Added Art
Parts:
- added H1, H2: ~, PCM_JLCPCB:Hole, 3mm, symbol PCM_JLCPCB-Manufacturing:Mounting Hole, 3mm, Via Stiched
Changed lines of the file:
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@@
+	)
+	(symbol
+		(lib_id "PCM_JLCPCB-Manufacturing:Mounting Hole, 3mm, Via Stiched")
+		(at 101.6 125.73 0)
+		(unit 1)
+		(exclude_from_sim no)
+		(in_bom yes)
+		(on_board yes)
+		(dnp no)
+		(fields_autoplaced yes)
+		(property "Reference" "H1"
+			(at 104.14 124.4599 0)
+			(effects
+				(font
+					(size 1.27 1.27)
+				)
+				(justify left)
+			)
+		)
+		(property "Value" "~"
+			(at 104.14 126.9999 0)
+			(effects
+				(font
+					(size 1.27 1.27)
+				)
+				(justify left)
+			)
+		)
+		(property "Footprint" "PCM_JLCPCB:Hole, 3mm"
+			(at 101.6 125.73 0)
+			(effects
+				(font
+					(size 1.27 1.27)
+				)
+				(hide yes)
+			)
+		)
+		(property "Datasheet" ""
+			(at 101.6 125.73 0)
+			(effects
+				(font
+					(size 1.27 1.27)
+				)
+				(hide yes)
+			)
+		)
+		(property "Description" ""
+			(at 101.6 125.73 0)
+			(effects
+				(font
+					(size 1.27 1.27)
+				)
+				(hide yes)
+			)
+		)
+		(pin "1"
+		)
+		(instances
+			(project ""
+				(path "/383cf046-a0a3-4840-8987-62617ca6a44c"
+					(reference "H1")
+					(unit 1)
+				)
+			)
+		)
 	)
 	(symbol
@@
 					(unit 1)
 				)
+			)
+		)
+	)
+	(symbol
+		(lib_id "PCM_JLCPCB-Manufacturing:Mounting Hole, 3mm, Via Stiched")
+		(at 101.6 120.65 0)
+		(unit 1)
+		(exclude_from_sim no)
+		(in_bom yes)
+		(on_board yes)
+		(dnp no)
+		(fields_autoplaced yes)
+		(property "Reference" "H2"
+			(at 104.14 119.3799 0)
+			(effects
+				(font
+					(size 1.27 1.27)
+				)
+				(justify left)
+			)
+		)
+		(property "Value" "~"
+			(at 104.14 121.9199 0)
+			(effects
+				(font
+					(size 1.27 1.27)
+				)
+				(justify left)
+			)
+		)
+		(property "Footprint" "PCM_JLCPCB:Hole, 3mm"
+			(at 101.6 120.65 0)
+			(effects
+				(font
+					(size 1.27 1.27)
+				)
+				(hide yes)
+			)
+		)
+		(property "Datasheet" ""
+			(at 101.6 120.65 0)
+			(effects
+				(font
+					(size 1.27 1.27)
+				)
+				(hide yes)
+			)
+		)
+		(property "Description" ""
+			(at 101.6 120.65 0)
+			(effects
+				(font
+					(size 1.27 1.27)
+				)
+				(hide yes)
+			)
+		)
+		(pin "1"
+		)
+		(instances
+			(project "PHMKeychain"
+				(path "/383cf046-a0a3-4840-8987-62617ca6a44c"
+					(reference "H2")
+					(unit 1)
+				)
